File: Board/Amplifier/Amplifier.sch (KiCad schematic (older format))
At the start: 11 parts

Commit message: Finished calculations
Parts:
- 1.6k: value R -> 800R
- R?: value 4R -> 6R
- R?: value 1R -> 0.6R
- R?: value 9.1k -> 21k
Other:
- moved on the sheet: C?
Changed lines of the file:
@@
 P 5150 2500
 F 0 "R?" H 5220 2546 50  0000 L CNN
-F 1 "4R" H 5220 2455 50  0000 L CNN
+F 1 "6R" H 5220 2455 50  0000 L CNN
 F 2 "" V 5080 2500 50  0001 C CNN
 F 3 "~" H 5150 2500 50  0001 C CNN
@@
 P 5150 3200
 F 0 "R?" H 5220 3246 50  0000 L CNN
-F 1 "1R" H 5220 3155 50  0000 L CNN
+F 1 "0.6R" H 5220 3155 50  0000 L CNN
 F 2 "" V 5080 3200 50  0001 C CNN
 F 3 "~" H 5150 3200 50  0001 C CNN
@@
 P 4850 3200
 F 0 "1.6k" H 4920 3246 50  0000 L CNN
-F 1 "R" H 4920 3155 50  0000 L CNN
+F 1 "800R" H 4920 3155 50  0000 L CNN
 F 2 "" V 4780 3200 50  0001 C CNN
 F 3 "~" H 4850 3200 50  0001 C CNN
@@
 P 4850 2500
 F 0 "R?" H 4920 2546 50  0000 L CNN
-F 1 "9.1k" H 4920 2455 50  0000 L CNN
+F 1 "21k" H 4920 2455 50  0000 L CNN
 F 2 "" V 4780 2500 50  0001 C CNN
 F 3 "~" H 4850 2500 50  0001 C CNN
@@
 	6150 2750 6150 3350
 Wire Wire Line
-	6150 3350 5450 3350
+	6150 3350 5550 3350
 $Comp
 L Device:CP C?
@@
 L Device:CP C?
 U 1 1 62455951
-P 5450 3200
-F 0 "C?" H 5568 3246 50  0000 L CNN
-F 1 "CP" H 5568 3155 50  0000 L CNN
-F 2 "" H 5488 3050 50  0001 C CNN
-F 3 "~" H 5450 3200 50  0001 C CNN
-	1    5450 3200
-	1    0    0    -1
-$EndComp
-Connection ~ 5450 3350
-Wire Wire Line
-	5450 3350 5150 3350
-Wire Wire Line
-	5450 3050 5150 3050
+P 5550 3200
+F 0 "C?" H 5668 3246 50  0000 L CNN
+F 1 "CP" H 5668 3155 50  0000 L CNN
+F 2 "" H 5588 3050 50  0001 C CNN
+F 3 "~" H 5550 3200 50  0001 C CNN
+	1    5550 3200
+	1    0    0    -1
+$EndComp
 Connection ~ 5150 3050
+Connection ~ 5550 3350
+Wire Wire Line
+	5150 3350 5550 3350
+Wire Wire Line
+	5150 3050 5550 3050
 $EndSCHEMATC
