File: Board/Amplifier/Amplifier.kicad_sch (KiCad schematic)
At the start: 22 parts, among them J1 Conn_01x02, J2 Conn_01x02, J3 AudioJack3, Q1 2SD2390

Commit message: Board design started
Parts:
- removed D1: B40R, Diode_THT:Diode_Bridge_Round_D9.0mm, symbol Diode_Bridge:B40R
- added D1: KBU8M, Diode_THT:Diode_Bridge_Vishay_KBU, symbol Diode_Bridge:KBU8M
- J1, J2: footprint (none) -> Amplifier Footprints:TB005-762-02BE
- J3: footprint (none) -> Connector_Audio:Jack_3.5mm_CUI_SJ1-3523N_Horizontal
- R2: footprint (none) -> Package_TO_SOT_THT:TO-247-2_Horizontal_TabUp
- R3: footprint (none) -> Package_TO_SOT_THT:TO-220-2_Horizontal_TabUp
- TP1, TP2, TP3, TP4, TP5, TP6: footprint (none) -> Connector_Wire:SolderWire-1sqmm_1x01_D1.4mm_OD3.9mm
Connections:
- net GND: now also D1.4 (-)
- net at F1.1: now also D1.1 (+)
- net at J1.1 (Pin_1): now also D1.2
- net at J1.2 (Pin_2): now also D1.3
Changed lines of the file:
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@@
       (effects (font (size 1.27 1.27)) (justify left))
     )
-    (property "Footprint" "" (id 2) (at 141.732 85.09 90)
+    (property "Footprint" "Package_TO_SOT_THT:TO-247-2_Horizontal_TabUp" (id 2) (at 141.732 85.09 90)
       (effects (font (size 1.27 1.27)) hide)
     )
@@
       (effects (font (size 1.27 1.27)) (justify left))
     )
-    (property "Footprint" "" (id 2) (at 141.732 125.73 90)
+    (property "Footprint" "Package_TO_SOT_THT:TO-220-2_Horizontal_TabUp" (id 2) (at 141.732 125.73 90)
       (effects (font (size 1.27 1.27)) hide)
     )
@@
     (pin "2")
   )
-  (symbol (lib_id "Diode_Bridge:B40R") (at 66.04 35.56 0) (unit 1)
-    (in_bom yes) (on_board yes)
-    (property "Reference" "D1" (id 0) (at 74.7776 34.3916 0)
-      (effects (font (size 1.27 1.27)) (justify left))
-    )
-    (property "Value" "B40R" (id 1) (at 74.7776 36.703 0)
-      (effects (font (size 1.27 1.27)) (justify left))
-    )
-    (property "Footprint" "Diode_THT:Diode_Bridge_Round_D9.0mm" (id 2) (at 69.85 32.385 0)
-      (effects (font (size 1.27 1.27)) (justify left) hide)
-    )
-    (property "Datasheet" "https://diotec.com/tl_files/diotec/files/pdf/datasheets/b40r.pdf" (id 3) (at 66.04 35.56 0)
-      (effects (font (size 1.27 1.27)) hide)
-    )
-    (pin "1")
-    (pin "2")
-    (pin "3")
-    (pin "4")
-  )
   (symbol (lib_id "Connector_Generic:Conn_01x02") (at 34.29 36.83 180) (unit 1)
     (in_bom yes) (on_board yes)
@@
       (effects (font (size 1.27 1.27)) (justify left))
     )
-    (property "Footprint" "" (id 2) (at 34.29 36.83 0)
+    (property "Footprint" "Amplifier Footprints:TB005-762-02BE" (id 2) (at 34.29 36.83 0)
       (effects (font (size 1.27 1.27)) hide)
     )
@@
       (effects (font (size 1.27 1.27)) (justify left))
     )
-    (property "Footprint" "" (id 2) (at 196.85 101.6 0)
+    (property "Footprint" "Amplifier Footprints:TB005-762-02BE" (id 2) (at 196.85 101.6 0)
       (effects (font (size 1.27 1.27)) hide)
     )
@@
       (effects (font (size 1.27 1.27)) (justify left))
     )
-    (property "Footprint" "" (id 2) (at 143.51 121.92 0)
+    (property "Footprint" "Connector_Wire:SolderWire-1sqmm_1x01_D1.4mm_OD3.9mm" (id 2) (at 143.51 121.92 0)
       (effects (font (size 1.27 1.27)) hide)
     )
@@
       (effects (font (size 1.27 1.27)) (justify left))
     )
-    (property "Footprint" "" (id 2) (at 118.11 35.56 0)
+    (property "Footprint" "Connector_Wire:SolderWire-1sqmm_1x01_D1.4mm_OD3.9mm" (id 2) (at 118.11 35.56 0)
       (effects (font (size 1.27 1.27)) hide)
     )
@@
       (effects (font (size 1.27 1.27)) (justify right))
     )
-    (property "Footprint" "" (id 2) (at 161.29 129.54 0)
+    (property "Footprint" "Connector_Wire:SolderWire-1sqmm_1x01_D1.4mm_OD3.9mm" (id 2) (at 161.29 129.54 0)
       (effects (font (size 1.27 1.27)) hide)
     )
@@
     (property "Reference" "J3" (id 0) (at 95.885 96.6302 0))
     (property "Value" "AudioJack3" (id 1) (at 95.885 99.1671 0))
-    (property "Footprint" "" (id 2) (at 97.79 104.14 0)
+    (property "Footprint" "Connector_Audio:Jack_3.5mm_CUI_SJ1-3523N_Horizontal" (id 2) (at 97.79 104.14 0)
       (effects (font (size 1.27 1.27)) hide)
     )
@@
     (property "Reference" "TP3" (id 0) (at 132.588 92.1852 90))
     (property "Value" "TestPoint" (id 1) (at 132.588 94.7221 90))
-    (property "Footprint" "" (id 2) (at 135.89 91.44 0)
+    (property "Footprint" "Connector_Wire:SolderWire-1sqmm_1x01_D1.4mm_OD3.9mm" (id 2) (at 135.89 91.44 0)
       (effects (font (size 1.27 1.27)) hide)
     )
@@
       (effects (font (size 1.27 1.27)) (justify left))
     )
-    (property "Footprint" "" (id 2) (at 129.54 35.56 0)
+    (property "Footprint" "Connector_Wire:SolderWire-1sqmm_1x01_D1.4mm_OD3.9mm" (id 2) (at 129.54 35.56 0)
       (effects (font (size 1.27 1.27)) hide)
     )
@@
     (pin "1")
   )
+  (symbol (lib_id "Diode_Bridge:KBU8M") (at 66.04 35.56 0) (unit 1)
+    (in_bom yes) (on_board yes) (fields_autoplaced)
+    (property "Reference" "D1" (id 0) (at 75.1001 32.8509 0))
+    (property "Value" "KBU8M" (id 1) (at 75.1001 35.3878 0))
+    (property "Footprint" "Diode_THT:Diode_Bridge_Vishay_KBU" (id 2) (at 69.85 32.385 0)
+      (effects (font (size 1.27 1.27)) (justify left) hide)
+    )
+    (property "Datasheet" "http://www.vishay.com/docs/88656/kbu8.pdf" (id 3) (at 66.04 35.56 0)
+      (effects (font (size 1.27 1.27)) hide)
+    )
+    (pin "1")
+    (pin "2")
+    (pin "3")
+    (pin "4")
+  )
   (symbol (lib_id "Device:R") (at 163.83 105.41 0) (unit 1)
     (in_bom yes) (on_board yes) (fields_autoplaced)
@@
       (effects (font (size 1.27 1.27)) (justify left))
     )
-    (property "Footprint" "" (id 2) (at 143.51 101.6 0)
+    (property "Footprint" "Connector_Wire:SolderWire-1sqmm_1x01_D1.4mm_OD3.9mm" (id 2) (at 143.51 101.6 0)
       (effects (font (size 1.27 1.27)) hide)
     )
@@
       (reference "C5") (unit 1) (value "100uF") (footprint "Capacitor_THT:CP_Radial_D12.5mm_P5.00mm")
     )
-    (path "/00000000-0000-0000-0000-00006219e3aa"
-      (reference "D1") (unit 1) (value "B40R") (footprint "Diode_THT:Diode_Bridge_Round_D9.0mm")
+    (path "/b88bfddc-74f8-492d-9fc6-6d986ac697d6"
+      (reference "D1") (unit 1) (value "KBU8M") (footprint "Diode_THT:Diode_Bridge_Vishay_KBU")
     )
     (path "/ef759f55-1234-45ec-aff8-33a9d20e6539"
@@
     )
     (path "/00000000-0000-0000-0000-00006219fbe1"
-      (reference "J1") (unit 1) (value "Conn_01x02") (footprint "")
+      (reference "J1") (unit 1) (value "Conn_01x02") (footprint "Amplifier Footprints:TB005-762-02BE")
     )
     (path "/00000000-0000-0000-0000-0000621a8bb2"
-      (reference "J2") (unit 1) (value "Conn_01x02") (footprint "")
+      (reference "J2") (unit 1) (value "Conn_01x02") (footprint "Amplifier Footprints:TB005-762-02BE")
     )
     (path "/926dd5e8-4411-46aa-adcf-c2510818230e"
-      (reference "J3") (unit 1) (value "AudioJack3") (footprint "")
+      (reference "J3") (unit 1) (value "AudioJack3") (footprint "Connector_Audio:Jack_3.5mm_CUI_SJ1-3523N_Horizontal")
     )
     (path "/00000000-0000-0000-0000-00006244f8e5"
@@
     )
     (path "/00000000-0000-0000-0000-00006219995f"
-      (reference "R2") (unit 1) (value "6R") (footprint "")
+      (reference "R2") (unit 1) (value "6R") (footprint "Package_TO_SOT_THT:TO-247-2_Horizontal_TabUp")
     )
     (path "/00000000-0000-0000-0000-00006219a661"
-      (reference "R3") (unit 1) (value "0.6R") (footprint "")
+      (reference "R3") (unit 1) (value "0.6R") (footprint "Package_TO_SOT_THT:TO-220-2_Horizontal_TabUp")
     )
     (path "/cc3a14f0-3bf3-4424-bb7d-a11f3f663c0b"
@@
     )
     (path "/695694ae-dbf5-42b8-8351-e1e7a942efe4"
-      (reference "TP1") (unit 1) (value "TestPoint") (footprint "")
+      (reference "TP1") (unit 1) (value "TestPoint") (footprint "Connector_Wire:SolderWire-1sqmm_1x01_D1.4mm_OD3.9mm")
     )
     (path "/b2e3525f-4fff-490d-8d72-d5045f77bcec"
-      (reference "TP2") (unit 1) (value "TestPoint") (footprint "")
+      (reference "TP2") (unit 1) (value "TestPoint") (footprint "Connector_Wire:SolderWire-1sqmm_1x01_D1.4mm_OD3.9mm")
     )
     (path "/9bcd9039-2c83-4d98-b6d8-803619ea0d1e"
-      (reference "TP3") (unit 1) (value "TestPoint") (footprint "")
+      (reference "TP3") (unit 1) (value "TestPoint") (footprint "Connector_Wire:SolderWire-1sqmm_1x01_D1.4mm_OD3.9mm")
     )
     (path "/e9bb1af2-98ce-47b4-8b23-f166931d33b4"
-      (reference "TP4") (unit 1) (value "TestPoint") (footprint "")
+      (reference "TP4") (unit 1) (value "TestPoint") (footprint "Connector_Wire:SolderWire-1sqmm_1x01_D1.4mm_OD3.9mm")
     )
     (path "/5ea58044-22f0-4d3b-9d94-1e76371692bb"
-      (reference "TP5") (unit 1) (value "TestPoint") (footprint "")
+      (reference "TP5") (unit 1) (value "TestPoint") (footprint "Connector_Wire:SolderWire-1sqmm_1x01_D1.4mm_OD3.9mm")
     )
     (path "/8de6c8d3-e4b0-4920-8ed4-c961f95d7b8f"
-      (reference "TP6") (unit 1) (value "TestPoint") (footprint "")
-    )
-  )
+      (reference "TP6") (unit 1) (value "TestPoint") (footprint "Connector_Wire:SolderWire-1sqmm_1x01_D1.4mm_OD3.9mm")
+    )
+  )
